Commit message: Update goliath.urdf.xacro

File: goliath_controller/description/urdf/goliath.urdf.xacro (robot description, xacro)
@@ -7,7 +7,9 @@
  <!-- Import goliath gripper macro -->
   <xacro:include filename="$(find gripper_description)/urdf/gripper.xacro"/>
-  <!-- create link fixed to the "world" -->
-  <link name="world"/>
+  <!-- create link fixed to the "world"
+  <link name="world"/> -->
   <xacro:goliath_description/>
+  <!-- Import goliath slider ros2_control description -->
+  <xacro:include filename="$(find base_link_linear_controller)/ros2_control/base_link_linear.ros2_control.xacro" />
   <!-- Import goliath ros2_control description -->
   <xacro:include filename="$(find goliath_controller)/ros2_control/goliath.ros2_control.xacro" />
