Commit message: Update goliath.ros2_control.xacro

File: goliath_controller/description/ros2_control/goliath.ros2_control.xacro (robot description, xacro)
@@ -138,4 +138,23 @@
       </joint>
     </ros2_control>
+    <ros2_control name="${name}_base" type="system">
+        <hardware>
+           <plugin>base_link_linear_controller/RobotSystem</plugin>
+           <param name="position1_joint_name">slider_11</param>
+           <param name="loop_rate">50</param>
+           <param name="device">/dev/ttyACM0</param>
+           <param name="baud_rate">115200</param>
+           <param name="timeout">1000</param>
+        </hardware>
+        <joint name="slider_11">
+           <command_interface name="position">
+             <param name="min">${-2*pi}</param>
+             <param name="max">${2*pi}</param>
+           </command_interface>
+           <state_interface name="position">
+             <param name="initial_value">0.0</param>
+           </state_interface>
+        </joint>
+   </ros2_control>
   </xacro:macro>
 </robot>

Commit message: Update goliath_controller pkg

File: goliath_controller/description/ros2_control/goliath.ros2_control.xacro (robot description, xacro)
@@ -109,33 +109,4 @@
       </sensor> -->
     </ros2_control>
-    <ros2_control name="${name}_gripper" type="system">
-      <hardware>
-        <plugin>gripper_controller/RobotSystem</plugin>
-        <param name="position1_joint_name">slider_22</param>
-        <param name="position2_joint_name">slider_23</param>
-        <param name="loop_rate">50</param>
-        <param name="device">/dev/ttyACM0</param>
-        <param name="baud_rate">115200</param>
-        <param name="timeout">1000</param>
-      </hardware>
-      <joint name="Slider 22">
-        <command_interface name="position">
-          <param name="min">${-2*pi}</param>
-          <param name="max">${2*pi}</param>
-        </command_interface>
-        <state_interface name="position">
-          <param name="initial_value">0.0</param>
-        </state_interface>
-      </joint>
-      <joint name="Slider 23">
-        <command_interface name="position">
-          <param name="min">${-2*pi}</param>
-          <param name="max">${2*pi}</param>
-        </command_interface>
-        <state_interface name="position">
-          <param name="initial_value">0.0</param>
-        </state_interface>
-      </joint>
-    </ros2_control>
     <ros2_control name="${name}_base" type="system">
         <hardware>

File: goliath_controller/description/urdf/base_link_linear.xacro (robot description, xacro)
@@ -4,5 +4,4 @@
 <xacro:include filename="$(find goliath_controller)/urdf/base_link_linear.trans" />
 <xacro:include filename="$(find goliath_controller)/urdf/base_link_linear.gazebo" />
-<xacro:include filename="$(find goliath_controller)/ros2_control/base_link_linear.ros2_control.xacro" />
 <link name="base_link">
   <visual>

File: goliath_controller/description/urdf/goliath.urdf.xacro (robot description, xacro)
@@ -10,6 +10,4 @@
   <link name="world"/> -->
   <xacro:goliath_description/>
-  <!-- Import goliath slider ros2_control description -->
-  <xacro:include filename="$(find goliath_controller)/ros2_control/base_link_linear.ros2_control.xacro" />
   <!-- Import goliath ros2_control description -->
   <xacro:include filename="$(find goliath_controller)/ros2_control/goliath.ros2_control.xacro" />

Commit message: Add files via upload

File: goliath_controller/description/ros2_control/goliath.ros2_control.xacro (robot description, xacro)
@@ -2,5 +2,5 @@
 <robot xmlns:xacro="http://www.ros.org/wiki/xacro">
   <xacro:macro name="goliath_ros2_control" params="name">
-    <ros2_control name="${name}_arm" type="system">
+    <ros2_control name="arm" type="system">
       <hardware>
         <plugin>goliath_controller/RobotSystem</plugin>
@@ -11,6 +11,7 @@
         <param name="position5_joint_name">position5_joint</param>
         <param name="position6_joint_name">position6_joint</param>
+        <param name="position7_joint_name">position7_joint</param>
         <param name="loop_rate">50</param>
-        <param name="device">/dev/ttyACM0</param>
+        <param name="device">/dev/ttyUSB0</param>
         <param name="baud_rate">115200</param>
         <param name="timeout">1000</param>
@@ -100,4 +101,13 @@
         <state_interface name="velocity"/>
       </joint>
+      <joint name="slider_11">
+         <command_interface name="position">
+           <param name="min">${0.455}</param>
+           <param name="max">${-0.455}</param>
+         </command_interface>
+         <state_interface name="position">
+           <param name="initial_value">0.0</param>
+         </state_interface>
+      </joint>
       <!-- <sensor name="tcp_fts_sensor">
         <state_interface name="force.x"/>
@@ -109,52 +119,4 @@
       </sensor> -->
     </ros2_control>
-    <ros2_control name="${name}_gripper" type="system">
-      <hardware>
-        <plugin>gripper_controller/RobotSystem</plugin>
-        <param name="position1_joint_name">slider_22</param>
-        <param name="position2_joint_name">slider_23</param>
-        <param name="loop_rate">50</param>
-        <param name="device">/dev/ttyACM0</param>
-        <param name="baud_rate">115200</param>
-        <param name="timeout">1000</param>
-      </hardware>
-      <joint name="Slider 22">
-        <command_interface name="position">
-          <param name="min">${-2*pi}</param>
-          <param name="max">${2*pi}</param>
-        </command_interface>
-        <state_interface name="position">
-          <param name="initial_value">0.0</param>
-        </state_interface>
-      </joint>
-      <joint name="Slider 23">
-        <command_interface name="position">
-          <param name="min">${-2*pi}</param>
-          <param name="max">${2*pi}</param>
-        </command_interface>
-        <state_interface name="position">
-          <param name="initial_value">0.0</param>
-        </state_interface>
-      </joint>
-    </ros2_control>
-    <ros2_control name="${name}_base" type="system">
-        <hardware>
-           <plugin>base_link_linear_controller/RobotSystem</plugin>
-           <param name="position1_joint_name">slider_11</param>
-           <param name="loop_rate">50</param>
-           <param name="device">/dev/ttyACM0</param>
-           <param name="baud_rate">115200</param>
-           <param name="timeout">1000</param>
-        </hardware>
-        <joint name="slider_11">
-           <command_interface name="position">
-             <param name="min">${-2*pi}</param>
-             <param name="max">${2*pi}</param>
-           </command_interface>
-           <state_interface name="position">
-             <param name="initial_value">0.0</param>
-           </state_interface>
-        </joint>
-   </ros2_control>
   </xacro:macro>
 </robot>
