Commit message: Update goliath_description.urdf.xacro

File: ros2_control_demo_description/goliath/urdf/goliath_description.urdf.xacro (robot description, xacro)
@@ -76,5 +76,5 @@
   <!-- joints - main serial chain -->
   <joint name="joint_1" type="revolute">
-    <parent link="base_link"/>
+    <parent link="arm_base_link"/>
     <child link="link_1"/>
     <origin xyz="0 0 0.104" rpy="0 0 0"/>

Commit message: Update goliath_description.urdf.xacro

File: ros2_control_demo_description/goliath/urdf/goliath_description.urdf.xacro (robot description, xacro)
@@ -5,5 +5,5 @@
   <xacro:include filename="$(find ros2_control_demo_description)/goliath/urdf/inc/create_link.xacro"/>
   <xacro:create_link
-      link_name="base_link"
+      link_name="arm_base_link"
       xyz_offset="0 0 0"
       rpy_offset="0 0 0"
@@ -68,8 +68,8 @@
       mesh_name="tool_base"
   />
-  <joint name="base_joint" type="fixed">
-    <parent link="world"/>
-    <child link="base_link"/>
-    <origin xyz="0 0 0" rpy="0 0 0"/>
+  <joint name="arm_base_joint" type="fixed">
+    <parent link="platform"/>
+    <child link="arm_base_link"/>
+    <origin xyz="0 0 0.09" rpy="0 0 0"/>
     <axis xyz="0 0 1"/>
   </joint>

Commit message: Update goliath_description.urdf.xacro

File: ros2_control_demo_description/goliath/urdf/goliath_description.urdf.xacro (robot description, xacro)
@@ -138,4 +138,9 @@
     <origin xyz="-0.0038 0.005 0.017" rpy="0 0 0"/>
   </joint>
+  <joint name="joint_powebox" type="fixed">
+    <parent link="link_2"/>
+    <child link="power_box"/>
+    <origin xyz="-0.276 0 -0.057" rpy="0 1.5775 0"/>
+  </joint>
 </xacro:macro>
 </robot>

Commit message: Add files via upload

File: ros2_control_demo_description/goliath/urdf/goliath_description.urdf.xacro (robot description, xacro)
@@ -60,20 +60,23 @@
       mesh_name="tool_connector"
   />
-<xacro:create_link
-      link_name="tool_connector"
-      xyz_offset="-0.0036 0.0053 0.0176"
-      rpy_offset="0 0 0"
+  <!--
+  <xacro:create_link
+      link_name="weapon"
+      xyz_offset="0.00 0.16 0.00"
+      rpy_offset="0 0 1.5775"
       material="silver"
       mesh_package="ros2_control_demo_description/goliath"
-      mesh_name="tool_base"
+      mesh_name="weapon2"
   />
-<xacro:create_link
+  -->
+  <xacro:create_link
       link_name="power_box"
       xyz_offset="0 0 0"
-      rpy_offset="0 0 0"
+      rpy_offset="0 1.5775 0"
       material="silver"
       mesh_package="ros2_control_demo_description/goliath"
       mesh_name="powerbox"
   />
+  <!-- ARM                                          -->
   <joint name="arm_base_joint" type="fixed">
     <parent link="platform"/>
@@ -125,21 +128,22 @@
     <limit effort="1000.0" lower="${-pi}" upper="${pi}" velocity="2.5"/>
   </joint>
-  <joint name="joint_tool_connector_frame" type="fixed">
-    <parent link="link_6"/>
-    <child link="tool_connector"/>
-    <origin xyz="0 0 0" rpy="0 0 0"/>
-  </joint>
   <!-- +++++++++++++++++++++++++++++++++++++++++++++++++++++++++++++++++++++++++++++++++++++++++
        joints for the tool - softgripper
        +++++++++++++++++++++++++++++++++++++++++++++++++++++++++++++++++++++++++++++++++++++++++ -->
-  <joint name="joint_connector_frame" type="fixed">
-    <parent link="tool_connector"/>
+  <joint name="joint_tool_connector_frame" type="fixed">
+    <parent link="link_6"/>
     <child link="tool_base"/>
-    <origin xyz="-0.0038 0.005 0.017" rpy="0 0 0"/>
+    <origin xyz="0 0 0.017" rpy="0 0 ${pi/2}"/>
   </joint>
-  <joint name="joint_powebox" type="fixed">
-    <parent link="link_2"/>
+<!--  <joint name="joint_weapon" type="fixed">
+    <parent link="tool_base"/>
+    <child link="weapon"/>
+    <origin xyz="0 0 0" rpy="0 0 0"/>
+  </joint>
+-->
+  <joint name="joint_powerbox" type="fixed">
+    <parent link="link_1"/>
     <child link="power_box"/>
-    <origin xyz="-0.276 0 -0.057" rpy="0 1.5775 0"/>
+    <origin xyz="0 -0.002 -0.108" rpy="${pi/2} ${-pi/2} 0"/>
   </joint>
 </xacro:macro>
