Commit message: Add files via upload

File: base_link_linear_controller/description/ros2_control/base_link_linear.ros2_control.xacro (robot description, xacro)
@@ -2,10 +2,10 @@
 <robot xmlns:xacro="http://www.ros.org/wiki/xacro">
  <xacro:macro name="base_link_linear_ros2_control" params="name">
-   <ros2_control name="${name}_base" type="system">
+ <ros2_control name="${name}" type="system">
         <hardware>
            <plugin>base_link_linear_controller/RobotSystem</plugin>
            <param name="position1_joint_name">slider_11</param>
            <param name="loop_rate">50</param>
-           <param name="device">/dev/ttyACM0</param>
+           <param name="device">/dev/ttyUSB0</param>
            <param name="baud_rate">115200</param>
            <param name="timeout">1000</param>
@@ -13,6 +13,6 @@
         <joint name="slider_11">
            <command_interface name="position">
-             <param name="min">${-2*pi}</param>
-             <param name="max">${2*pi}</param>
+             <param name="min">${-0.455}</param>
+             <param name="max">${0.455}</param>
            </command_interface>
            <state_interface name="position">
@@ -20,5 +20,5 @@
            </state_interface>
         </joint>
-   </ros2_control>
-  </xacro:macro>
+  </ros2_control>
+ </xacro:macro>
 </robot>
