Commit message: Add files via upload

File: base_link_linear_controller/description/urdf/base_link_linear.xacro (robot description, xacro)
@@ -5,5 +5,6 @@
 <xacro:include filename="$(find base_link_linear_controller)/urdf/base_link_linear.gazebo" />
 <xacro:include filename="$(find base_link_linear_controller)/ros2_control/base_link_linear.ros2_control.xacro" />
-<link name="base_link">
+<xacro:base_link_linear_ros2_control name="base_link_linear_ros2_control"/>
+<link name="base_link_linear">
   <visual>
     <origin xyz="0 0 0" rpy="0 0 0"/>
@@ -17,4 +18,18 @@
     <geometry>
       <mesh filename="file://$(find base_link_linear_description)/meshes/base_link.stl" scale="0.001 0.001 0.001"/>
+    </geometry>
+  </collision>
+</link>
+<link name="unilidar_imu_initial">
+ <visual>
+ <origin xyz="0 0 0" rpy="0 0 0"/>
+ <geometry>
+    <cylinder radius="0.04" length="0.06"/>
+ </geometry>
+    <material name="blue"/>
+ </visual>
+  <collision>
+    <geometry>
+      <cylinder radius="0.04" length="0.06"/>
     </geometry>
   </collision>
@@ -109,5 +124,5 @@
     <origin xyz="-0.002356 -0.0 -0.03" rpy="0 0 0"/>
     <geometry>
-      <mesh filename="file://$(find base_link_linear_description)/meshes/platform_v2_1.stl" scale="0.001 0.001 0.001"/>
+      <mesh filename="file://$(find base_link_linear_description)/meshes/platform.stl" scale="0.001 0.001 0.001"/>
     </geometry>
     <material name="silver"/>
@@ -116,5 +131,5 @@
     <origin xyz="-0.002356 -0.0 -0.03" rpy="0 0 0"/>
     <geometry>
-      <mesh filename="file://$(find base_link_linear_description)/meshes/platform_v2_1.stl" scale="0.001 0.001 0.001"/>
+      <mesh filename="file://$(find base_link_linear_description)/meshes/platform.stl" scale="0.001 0.001 0.001"/>
     </geometry>
   </collision>
@@ -172,18 +187,18 @@
 <joint name="Rigid 8" type="fixed">
   <origin xyz="0.122356 0.498326 0.058" rpy="0 0 0"/>
-  <parent link="base_link"/>
+  <parent link="base_link_linear"/>
   <child link="rail_2_v1_1"/>
 </joint>
 <joint name="Rigid 9" type="fixed">
   <origin xyz="-0.117644 0.498326 0.058" rpy="0 0 0"/>
-  <parent link="base_link"/>
+  <parent link="base_link_linear"/>
   <child link="rail_1_v1_1"/>
 </joint>
 <joint name="slider_11" type="prismatic">
   <origin xyz="0.002356 0.0 0.03" rpy="0 0 0"/>
-  <parent link="base_link"/>
+  <parent link="base_link_linear"/>
   <child link="platform"/>
   <axis xyz="0.0 1.0 0.0"/>
-  <limit upper="0.34" lower="-0.35" effort="100" velocity="100"/>
+  <limit upper="0.455" lower="-0.455" effort="100" velocity="100"/>
 </joint>
 <joint name="Rigid 12" type="fixed">
@@ -197,3 +212,8 @@
   <child link="block2_1"/>
 </joint>
+<joint name="Rigid 15" type="fixed">
+  <origin xyz="0.0 0.65 0.07" rpy="0 0 -0.2"/>
+  <parent link="base_link_linear"/>
+  <child link="unilidar_imu_initial"/>
+</joint>
 </robot>
